File: IntegratedMotorController_pcb/DARPA_MCTR.kicad_pcb (KiCad board)
At the start: 4 copper layers, 52 x 51 mm, 100 parts, among them IC2 TCAN3413DR, IC3 FM24CL64B-GTR, J1 USB_B_Micro, J2 436500301, J3 436500301, J4 436500401, J5 436500201, J8 436500201, J9 436500201, K1 TX2-12V-TH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

Commit message: new version 1.1
Parts:
- removed C33: 1u, Capacitor_SMD:C_0402_1005Metric
- removed D2: LED, LED_SMD:LED_0603_1608Metric
- removed R14: 27, Resistor_SMD:R_0402_1005Metric
- removed R24, R25, R26, R29: 10k, Resistor_SMD:R_0603_1608Metric
- removed R27: 4.7k, Resistor_SMD:R_0603_1608Metric
- removed TP3: SWCLK, TestPoint:TestPoint_Pad_1.0x1.0mm
- removed TP4: SWD, TestPoint:TestPoint_Pad_1.0x1.0mm
- removed U6: TPS2121RUXT, DARPA:RUX0012A
- added C4: UCD1V101MCL6GS, DARPA:PCAP_6.3x7.7-ELECT_NCA, F.Cu at (103.5, 81.0)
- added CR1: SMAJ13A, DARPA:SMASeries_LTF, F.Cu at (102.7, 86.5)
- added CR2: B340A-13-F, DARPA:DIODE_SODB340_2P92X4P6_DIO, F.Cu at (108.2, 73.8)
- added GND: 5V5, TestPoint:TestPoint_Pad_1.0x1.0mm, F.Cu at (109.5, 119.0)
- added J6: BM03B-SRSS-TBLFSN, DARPA:CONN_BM03B-SRSS-TBLFSN_JST, F.Cu at (98.5, 117.2)
- R23: value 33.2k -> 4.7k
- moved R23 16.9 mm to (107.1, 100.0), turned to 0 degrees
- moved D3 8.00 mm to (106.8, 118.8), turned to 180 degrees
- moved C17 5.00 mm to (109.2, 82.8), turned to 0 degrees
- moved C20 4.42 mm to (109.2, 80.0), turned to -90 degrees
- moved R15 3.76 mm to (104.0, 118.8), turned to 0 degrees
- moved C1 3.55 mm to (105.5, 74.0), turned to 90 degrees
- moved C21 2.25 mm to (115.2, 77.0)
- moved C22 2.25 mm to (117.2, 72.5)
- moved C23 2.25 mm to (117.2, 74.5)
- moved L1 2.25 mm to (112.8, 73.5)
- moved R12 2.25 mm to (113.1, 80.8)
- moved R13 2.25 mm to (115.5, 79.4)
- moved VR1 2.25 mm to (112.5, 78.0)
- moved TP1 2.16 mm to (113.8, 119.0)
- moved TP2 2.16 mm to (111.5, 119.0)
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Connections:
- C20 pad 1: /BUCK2_IN -> +12V
- R23 pad 1: +12V -> /PGOOD
- R23 pad 2: Net-(U6-PR1) -> +3V3
- U3 pad 36: /POWER_SRC -> unconnected-(U3-GPIO24-Pad36)
- VR1 pad 3: /BUCK2_IN -> +12V
- VR1 pad 5: /BUCK2_IN -> +12V
Routing:
- net /POWER_SRC: track 28.7 -> 0.00 mm, vias 3 -> 0
- net /PGOOD: track 19.9 -> 28.3 mm
- net VBUS: track 2.11 -> 10.5 mm
- net Net-(U6-PR1): track 5.29 -> 0.00 mm
- net Net-(U3-RUN): track 66.8 -> 71.9 mm
- net GND: track 49.7 -> 53.7 mm, vias 52 -> 54
- net /SWD: track 17.8 -> 20.6 mm
- net /LED: track 14.9 -> 17.6 mm, vias 2 -> 0
- net /5V5_PREINA: track 33.8 -> 31.7 mm
- net +12V: track 6.53 -> 8.51 mm, vias 1 -> 6
- net Net-(U6-ILM): track 1.69 -> 0.00 mm
- net +3V3: track 58.8 -> 57.1 mm, vias 20 -> 18
- net Net-(R25-Pad2): track 1.50 -> 0.00 mm
- net Net-(D2-A): track 1.16 -> 0.00 mm
- net Net-(U6-SS): track 1.14 -> 0.00 mm
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- removed copper zone on F.Cu, net /BUCK2_IN
- removed copper zone on F.Cu, net VBUS
Other:
- board text added: "Alek - Rev 1.1 - 2026"
- board text added: "STATUS"
- board text removed: "Alek - Rev 1.0 - 2026"
- board text removed: "PWR"
- board text removed: "STAT"
