File: IntegratedMotorController_pcb/DARPA_MCTR.kicad_sch (KiCad schematic)
At the start: 100 parts, among them IC2 TCAN3413DR, IC3 FM24CL64B-GTR, J1 USB_B_Micro, J2 436500301, J3 436500301, J4 436500401, J5 436500201, J8 436500201, J9 436500201, K1 TX2-12V-TH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

Commit message: new version 1.1
Parts:
- removed C33: 1u, Capacitor_SMD:C_0402_1005Metric, symbol Device:C
- removed D2: LED, LED_SMD:LED_0603_1608Metric, symbol Device:LED
- removed R14: 27, Resistor_SMD:R_0402_1005Metric, symbol Device:R
- removed R24, R25, R26, R29: 10k, Resistor_SMD:R_0603_1608Metric, symbol Device:R_Small
- removed R27: 4.7k, Resistor_SMD:R_0603_1608Metric, symbol Device:R_Small
- removed TP4: SWD, TestPoint:TestPoint_Pad_1.0x1.0mm, symbol Connector:TestPoint
- removed U6: TPS2121RUXT, DARPA:RUX0012A, symbol DARPA:TPS2121RUXT
- added C4: UCD1V101MCL6GS, DARPA:PCAP_6.3x7.7-ELECT_NCA, symbol DARPA:UCD1V101MCL6GS
- added CR1: SMAJ13A, DARPA:SMASeries_LTF, symbol DARPA:SMAJ13A
- added CR2: B340A-13-F, DARPA:DIODE_SODB340_2P92X4P6_DIO, symbol DARPA:B340A-13-F
- added J6: BM03B-SRSS-TBLFSN, DARPA:CONN_BM03B-SRSS-TBLFSN_JST, symbol DARPA:BM03B-SRSS-TBLFSN
- R23: value 33.2k -> 4.7k; DPN 311-33.2KHRCT-ND -> 311-4.70KHRCT-ND; MPN RC0603FR-0733K2L -> RC0603FR-074K7L
- TP3: value SWCLK -> 5V5
Connections:
- net BUCK2_IN is gone; now on net +12V: C20.1, VR1.3 (VIN), VR1.5 (EN)
- net +12V: now also C4.1, CR1.1, CR2.1; no longer R23.1
- net +3V3: now also R23.2
- net GND: now also TP3.1, C4.2, CR1.2, J6.2, J6.4, J6.5
- net PGOOD: now also R23.1
- net SWCLK: now also J6.1; no longer TP3.1
- net SWD: now also J6.3
- net VBUS: now also CR2.2
- net POWER_SRC: no longer names the net of U3.36 (GPIO24)
- no-connect marks 19 -> 20
Other:
- note added: "I know this it a bad idea but i promise I will be carefull"
- note added: "JST debug connector"
- moved on the sheet: C5, R1, R2, SW2, U2

Commit message: Some cleanup and new stuff
Parts:
- C1, C17, C20: JLC (none) -> C440198
- C10, C8: JLC (none) -> C14445
- C11, C12, C13, C14, C15, C16, C18, C21, C24, C27, C28, C29, C32, C5, C6, C7, C9: JLC (none) -> C71629
- C19, C22, C23, C30, C31, C34: JLC (none) -> C441864
- C2, C25, C26, C3: JLC (none) -> C1548
- C4: JLC (none) -> C134220
- CR1: JLC (none) -> C5356038
- CR2: JLC (none) -> C85098
- D1: JLC (none) -> C9900174479
- D3: JLC (none) -> C9900202211
- IC2: JLC (none) -> C22433320
- IC3: JLC (none) -> C9829
- J1: JLC (none) -> C428495
- J6: JLC (none) -> C160389
- L1: JLC (none) -> C139481
- Q1: JLC (none) -> C20917
- R1, R11, R5: JLC (none) -> C11702
- R10, R12, R17, R18, R7, R8: JLC (none) -> C25804
- R13: JLC (none) -> C4089611
- R15, R3, R4: JLC (none) -> C25100
- R16, R19, R20, R21, R22, R23: JLC (none) -> C23162
- R6: JLC (none) -> C23254
- R9: JLC (none) -> C413486
- SW2, SW3: JLC (none) -> C79161
- U1: JLC (none) -> C48581090
- U2: JLC (none) -> C97521
- U3: JLC (none) -> C2040
- U4: JLC (none) -> C138706
- U5: JLC (none) -> C621395
- VR1: JLC (none) -> C138335
- Y1: JLC (none) -> C20625731
- Y2: JLC (none) -> C596863
